Commit message: camera_setting

File: src/camera_setting/urdf/camera.urdf.xacro (robot description, xacro)
@@ -1,17 +1,21 @@
 <?xml version="1.0"?>
 <robot xmlns:xacro="http://www.ros.org/wiki/xacro" name="firefighter">
-<xacro:arg name="parent" default="world"/>
+<xacro:property name="camera_roll" value="0.0" />
+<xacro:property name="camera_pitch" value="0.7853" />
+<xacro:property name="camera_yaw" value="0.7853" />
+<xacro:arg name="parent" default="base_link"/>
 <xacro:include filename="$(find camera_setting)/urdf/camera.xacro"/>
-<xacro:camera name="A" parent="$(arg parent)">
-	<origin xyz="10.0 10.0 10.0" rpy="0.0 0.0 0.0"/>
-</xacro:camera>
-<xacro:camera name="B" parent="$(arg parent)">
-	<origin xyz="-10.0 10.0 10.0" rpy="0.0 0.0 0.0"/>
-</xacro:camera>
-<xacro:camera name="C" parent="$(arg parent)">
-	<origin xyz="10.0 -10.0 10.0" rpy="0 0 0"/>
-</xacro:camera>
-<xacro:camera name="D" parent="$(arg parent)">
-	<origin xyz="-10.0 -10.0 10.0" rpy="0 0 0"/>
-</xacro:camera>
+<xacro:base/>
+<xacro:camera_link name="A" parent="$(arg parent)">
+	<origin xyz="2.5 2.5 2.5" rpy="${camera_roll} ${camera_pitch} ${3.1416 + camera_yaw}"/>
+</xacro:camera_link>
+<xacro:camera_link name="B" parent="$(arg parent)">
+	<origin xyz="-2.5 2.5 2.5" rpy="${camera_roll} ${camera_pitch} ${4.712 + camera_yaw}"/>
+</xacro:camera_link>
+<xacro:camera_link name="C" parent="$(arg parent)">
+	<origin xyz="2.5 -2.5 2.5" rpy="${camera_roll} ${camera_pitch} ${1.508 + camera_yaw}"/>
+</xacro:camera_link>
+<xacro:camera_link name="D" parent="$(arg parent)">
+	<origin xyz="-2.5 -2.5 2.5" rpy="${camera_roll} ${camera_pitch} ${camera_yaw}"/>
+</xacro:camera_link>
 </robot>

File: src/camera_setting/urdf/camera.xacro (robot description, xacro)
@@ -1,15 +1,50 @@
 <?xml version="1.0"?>
 <robot xmlns:xacro="http://www.ros.org/wiki/xacro" name="firefighter">
-<xacro:macro name="camera" params="name parent *origin">
-	<link name="camera_${name}_link">
+<xacro:macro name="base">
+	<link name="base_link">
 		<visual>
 			<origin xyz="0.0 0.0 0.0" rpy="0.0 0.0 0.0"/>
-		    <geometry>
-		        <box size="0.1 0.1 0.1" />
-		    </geometry>
+			<geometry>
+				<box size="0.1 0.1 0.1" />
+			</geometry>
 			<material name="rrr">
 				<color rgba="1.0 0.0 0 0.5"/>
 			</material>
 		</visual>
+		<collision>
+			<origin xyz="0 0 0" rpy="0 0 0"/>
+			<geometry>
+				<box size="0.1 0.1 0.1" />
+			</geometry>
+		</collision>
+		<inertial>
+			<mass value="0.001" />
+			<origin xyz="0 0 0" rpy="0 0 0" />
+			<inertia ixx="0.0001" ixy="0" ixz="0" iyy="0.0001" iyz="0" izz="0.0001" />
+		</inertial>
+	</link>
+</xacro:macro>
+<xacro:macro name="camera_link" params="name parent *origin">
+	<link name="camera_${name}_link">
+		<visual>
+			<origin xyz="0 0 0" rpy="0 0 0" />
+			<geometry>
+				<box size="0.1 0.1 0.1" />
+			</geometry>
+			<material name="grey">
+				<color rgba="0.2 0.2 0.2 1.0"/>
+			</material>
+		</visual>
+		<collision>
+			<origin xyz="0 0 0" rpy="0 0 0"/>
+			<geometry>
+				<box size="0.1 0.1 0.1" />
+			</geometry>
+		</collision>
+		<inertial>
+			<mass value="0.001" />
+			<origin xyz="0 0 0" rpy="0 0 0" />
+			<inertia ixx="0.0001" ixy="0" ixz="0" iyy="0.0001" iyz="0" izz="0.0001" />
+		</inertial>
 	</link>
 	<joint name="camera_${name}_joint" type="fixed">
@@ -19,43 +54,44 @@
 		<child link="camera_${name}_link"/>
 	</joint>
-  <gazebo reference="camera_${name}_link">
-    <sensor type="camera" name="camera1">
-      <update_rate>30.0</update_rate>
-      <camera name="head">
-        <horizontal_fov>1.3962634</horizontal_fov>
-        <image>
-          <width>800</width>
-          <height>800</height>
-          <format>R8G8B8</format>
-        </image>
-        <clip>
-          <near>0.02</near>
-          <far>300</far>
-        </clip>
-        <noise>
-          <type>gaussian</type>
-          <!-- Noise is sampled independently per pixel on each frame.
-               That pixel's noise value is added to each of its color
-               channels, which at that point lie in the range [0,1]. -->
-          <mean>0.0</mean>
-          <stddev>0.007</stddev>
-        </noise>
-      </camera>
-      <plugin name="camera_controller" filename="libgazebo_ros_camera.so">
-        <alwaysOn>true</alwaysOn>
-        <updateRate>0.0</updateRate>
-        <cameraName>rrbot/camera1</cameraName>
-        <imageTopicName>image_raw</imageTopicName>
-        <cameraInfoTopicName>camera_info</cameraInfoTopicName>
-        <frameName>sonar_link</frameName>
-        <hackBaseline>0.07</hackBaseline>
-        <distortionK1>0.0</distortionK1>
-        <distortionK2>0.0</distortionK2>
-        <distortionK3>0.0</distortionK3>
-        <distortionT1>0.0</distortionT1>
-        <distortionT2>0.0</distortionT2>
-      </plugin>
-    </sensor>
-  </gazebo>
+  	<gazebo reference="camera_${name}_link">
+		<sensor type="camera" name="camera_${name}">
+			<update_rate>30.0</update_rate>
+			<visualize>1</visualize>
+			<camera name="camera_${name}">
+				<horizontal_fov>1.3962634</horizontal_fov>
+				<image>
+					<width>800</width>
+					<height>800</height>
+					<format>R8G8B8</format>
+				</image>
+				<clip>
+					<near>0.02</near>
+					<far>300</far>
+				</clip>
+				<noise>
+					<type>gaussian</type>
+					<!-- Noise is sampled independently per pixel on each frame.
+						That pixel's noise value is added to each of its color
+						channels, which at that point lie in the range [0,1]. -->
+					<mean>0.0</mean>
+					<stddev>0.007</stddev>
+				</noise>
+			</camera>
+			<plugin name="camera_controller" filename="libgazebo_ros_camera.so">
+				<alwaysOn>true</alwaysOn>
+				<updateRate>0.0</updateRate>
+				<cameraName>rrbot/camera_${name}</cameraName>
+				<imageTopicName>image_raw</imageTopicName>
+				<cameraInfoTopicName>camera_info</cameraInfoTopicName>
+				<frameName>camera_${name}_link</frameName>
+				<hackBaseline>0.07</hackBaseline>
+				<distortionK1>0.0</distortionK1>
+				<distortionK2>0.0</distortionK2>
+				<distortionK3>0.0</distortionK3>
+				<distortionT1>0.0</distortionT1>
+				<distortionT2>0.0</distortionT2>
+			</plugin>
+		</sensor>
+	</gazebo>
 </xacro:macro>
 </robot>

Commit message: camera_setting modification

File: src/camera_setting/urdf/camera.urdf.xacro (robot description, xacro)
@@ -1,9 +1,12 @@
 <?xml version="1.0"?>
 <robot xmlns:xacro="http://www.ros.org/wiki/xacro" name="firefighter">
+<!--
 <xacro:property name="camera_roll" value="0.0" />
 <xacro:property name="camera_pitch" value="0.7853" />
 <xacro:property name="camera_yaw" value="0.7853" />
 <xacro:arg name="parent" default="base_link"/>
+-->
 <xacro:include filename="$(find camera_setting)/urdf/camera.xacro"/>
+<!--
 <xacro:base/>
 <xacro:camera_link name="A" parent="$(arg parent)">
@@ -19,3 +22,5 @@
 	<origin xyz="-2.5 -2.5 2.5" rpy="${camera_roll} ${camera_pitch} ${camera_yaw}"/>
 </xacro:camera_link>
+-->
+<xacro:camera_model name="A"/>
 </robot>

File: src/camera_setting/urdf/camera.xacro (robot description, xacro)
@@ -1,4 +1,5 @@
 <?xml version="1.0"?>
 <robot xmlns:xacro="http://www.ros.org/wiki/xacro" name="firefighter">
+<!--
 <xacro:macro name="base">
 	<link name="base_link">
@@ -25,6 +26,8 @@
 	</link>
 </xacro:macro>
-<xacro:macro name="camera_link" params="name parent *origin">
-	<link name="camera_${name}_link">
+-->
+<xacro:arg name="camera_name" default="A"/>
+<xacro:macro name="camera_model" params="name">
+	<link name="camera_link">
 		<visual>
 			<origin xyz="0 0 0" rpy="0 0 0" />
@@ -43,9 +46,18 @@
 		</collision>
 		<inertial>
-			<mass value="0.001" />
+			<mass value="0.1" />
 			<origin xyz="0 0 0" rpy="0 0 0" />
-			<inertia ixx="0.0001" ixy="0" ixz="0" iyy="0.0001" iyz="0" izz="0.0001" />
+			<inertia ixx="1" ixy="0" ixz="0" iyy="1" iyz="0" izz="1" />
 		</inertial>
 	</link>
+        <!-- set the model to be static -->
+        <gazebo>
+        	<static>true</static>
+	</gazebo>
+        <!-- set gravity of camera to zero -->
+        <!--gazebo reference="camera_link">
+        	<gravity>0 0 0</gravity>
+	</gazebo-->
+        <!--
 	<joint name="camera_${name}_joint" type="fixed">
 		<xacro:insert_block name="origin" />
@@ -54,5 +66,6 @@
 		<child link="camera_${name}_link"/>
 	</joint>
-  	<gazebo reference="camera_${name}_link">
+        -->
+  	<gazebo reference="camera_link">
 		<sensor type="camera" name="camera_${name}">
 			<update_rate>30.0</update_rate>
@@ -80,8 +93,8 @@
 			<plugin name="camera_controller" filename="libgazebo_ros_camera.so">
 				<alwaysOn>true</alwaysOn>
-				<updateRate>0.0</updateRate>
-				<cameraName>rrbot/camera_${name}</cameraName>
-				<imageTopicName>image_raw</imageTopicName>
-				<cameraInfoTopicName>camera_info</cameraInfoTopicName>
+				<updateRate>30.0</updateRate>
+				<cameraName>camera_${name}/name</cameraName>
+				<imageTopicName>/camera_${name}/image_raw</imageTopicName>
+				<cameraInfoTopicName>/camera_${name}/camera_info</cameraInfoTopicName>
 				<frameName>camera_${name}_link</frameName>
 				<hackBaseline>0.07</hackBaseline>
@@ -95,3 +108,4 @@
 	</gazebo>
 </xacro:macro>
+<xacro:camera_model name="$(arg camera_name)"/>
 </robot>
