Commit message: add color (hsv) detector

File: src/multi_view_plugin/urdf/camera.xacro (robot description, xacro)
@@ -1,110 +1,78 @@
 <?xml version="1.0"?>
-<robot xmlns:xacro="http://www.ros.org/wiki/xacro" name="firefighter">
-<!--
-<xacro:macro name="base">
-	<link name="base_link">
-		<visual>
-			<origin xyz="0.0 0.0 0.0" rpy="0.0 0.0 0.0"/>
-			<geometry>
-				<box size="0.1 0.1 0.1" />
-			</geometry>
-			<material name="rrr">
-				<color rgba="1.0 0.0 0 0.5"/>
-			</material>
-		</visual>
-		<collision>
-			<origin xyz="0 0 0" rpy="0 0 0"/>
-			<geometry>
-				<box size="0.1 0.1 0.1" />
-			</geometry>
-		</collision>
-		<inertial>
-			<mass value="0.001" />
-			<origin xyz="0 0 0" rpy="0 0 0" />
-			<inertia ixx="0.0001" ixy="0" ixz="0" iyy="0.0001" iyz="0" izz="0.0001" />
-		</inertial>
-	</link>
-</xacro:macro>
--->
-<xacro:arg name="camera_name" default="A"/>
-<xacro:macro name="camera_model" params="name">
-	<link name="camera_link">
-		<visual>
-			<origin xyz="0 0 0" rpy="0 0 0" />
-			<geometry>
-				<box size="0.1 0.1 0.1" />
-			</geometry>
-			<material name="grey">
-				<color rgba="0.2 0.2 0.2 1.0"/>
-			</material>
-		</visual>
-		<collision>
-			<origin xyz="0 0 0" rpy="0 0 0"/>
-			<geometry>
-				<box size="0.1 0.1 0.1" />
-			</geometry>
-		</collision>
-		<inertial>
-			<mass value="0.1" />
-			<origin xyz="0 0 0" rpy="0 0 0" />
-			<inertia ixx="1" ixy="0" ixz="0" iyy="1" iyz="0" izz="1" />
-		</inertial>
-	</link>
-        <!-- set the model to be static -->
-        <gazebo>
-        	<static>true</static>
-	</gazebo>
-        <!-- set gravity of camera to zero -->
-        <!--gazebo reference="camera_link">
-        	<gravity>0 0 0</gravity>
-	</gazebo-->
-        <!--
-	<joint name="camera_${name}_joint" type="fixed">
-		<xacro:insert_block name="origin" />
-		<axis xyz="0 1 0"/>
-		<parent link="${parent}"/>
-		<child link="camera_${name}_link"/>
-	</joint>
-        -->
-  	<gazebo reference="camera_link">
-		<sensor type="camera" name="camera_${name}">
-			<update_rate>30.0</update_rate>
-			<visualize>1</visualize>
-			<camera name="camera_${name}">
-				<horizontal_fov>1.3962634</horizontal_fov>
-				<image>
-					<width>800</width>
-					<height>800</height>
-					<format>R8G8B8</format>
-				</image>
-				<clip>
-					<near>0.02</near>
-					<far>300</far>
-				</clip>
-				<noise>
-					<type>gaussian</type>
-					<!-- Noise is sampled independently per pixel on each frame.
-						That pixel's noise value is added to each of its color
-						channels, which at that point lie in the range [0,1]. -->
-					<mean>0.0</mean>
-					<stddev>0.007</stddev>
-				</noise>
-			</camera>
-			<plugin name="camera_controller" filename="libgazebo_ros_camera.so">
-				<alwaysOn>true</alwaysOn>
-				<updateRate>30.0</updateRate>
-				<cameraName>camera_${name}/name</cameraName>
-				<imageTopicName>/camera_${name}/image_raw</imageTopicName>
-				<cameraInfoTopicName>/camera_${name}/camera_info</cameraInfoTopicName>
-				<frameName>camera_${name}_link</frameName>
-				<hackBaseline>0.07</hackBaseline>
-				<distortionK1>0.0</distortionK1>
-				<distortionK2>0.0</distortionK2>
-				<distortionK3>0.0</distortionK3>
-				<distortionT1>0.0</distortionT1>
-				<distortionT2>0.0</distortionT2>
-			</plugin>
-		</sensor>
-	</gazebo>
+<robot name="ball_tracker" xmlns:xacro="http://www.ros.org/wiki/xacro">
+  <xacro:arg name="camera_name" default="A"/>
+  <xacro:macro name="camera_model" params="name">
+    <link name="camera_link">
+      <visual>
+        <origin xyz="0 0 0" rpy="0 0 0" />
+	<geometry>
+	  <box size="0.1 0.1 0.1" />
+	</geometry>
+	<material name="grey">
+	  <color rgba="0.2 0.2 0.2 1.0"/>
+        </material>
+      </visual>
+      <collision>
+        <origin xyz="0 0 0" rpy="0 0 0"/>
+	<geometry>
+	  <box size="0.1 0.1 0.1" />
+	</geometry>
+      </collision>
+      <inertial>
+	<mass value="0.1" />
+	<origin xyz="0 0 0" rpy="0 0 0" />
+	<inertia ixx="1" ixy="0" ixz="0" iyy="1" iyz="0" izz="1" />
+      </inertial>
+    </link>
+    <!-- disable the gravity of camera -->
+    <gazebo reference="camera_link">
+      <gravity>false</gravity>
+    </gazebo>
+    <gazebo reference="camera_link">
+      <sensor type="camera" name="camera_${name}">
+	<update_rate>30.0</update_rate>
+	<visualize>1</visualize>
+	<camera name="camera_${name}">
+	  <horizontal_fov>1.3962634</horizontal_fov>
+          <image>
+	    <width>800</width>
+	    <height>800</height>
+	    <format>R8G8B8</format>
+	  </image>
+	  <clip>
+	    <near>0.02</near>
+	    <far>300</far>
+	  </clip>
+	  <noise>
+	    <type>gaussian</type>
+            <!-- Noise is sampled independently per pixel on each frame. That pixel's noise value is added to each of its color channels, which at that point lie in the range [0,1]. -->
+	    <mean>0.0</mean>
+	    <stddev>0.007</stddev>
+	  </noise>
+	</camera>
+	<plugin name="camera_controller" filename="libgazebo_ros_camera.so">
+          <alwaysOn>true</alwaysOn>
+	  <updateRate>30.0</updateRate>
+	  <cameraName>camera_${name}/name</cameraName>
+	  <imageTopicName>/camera_${name}/image_raw</imageTopicName>
+	  <cameraInfoTopicName>/camera_${name}/camera_info</cameraInfoTopicName>
+	  <frameName>camera_${name}_link</frameName>
+	  <hackBaseline>0.07</hackBaseline>
+	  <distortionK1>0.0</distortionK1>
+	  <distortionK2>0.0</distortionK2>
+	  <distortionK3>0.0</distortionK3>
+	  <distortionT1>0.0</distortionT1>
+	  <distortionT2>0.0</distortionT2>
+	</plugin>
+      </sensor>
+    </gazebo>
+    <gazebo>
+      <plugin filename="libball_tracker.so" name="ball_tracker_controller">
+        <camera_name>camera_${name}</camera_name>
+        <raw_topic>camera_${name}/image_raw</raw_topic>
+        <binary_topic>camera_${name}/image_filtered</binary_topic>
+        <cm_topic>camera_${name}/2D_tracking</cm_topic>
+      </plugin>
+    </gazebo>
 </xacro:macro>
 <xacro:camera_model name="$(arg camera_name)"/>
