Commit message: backup before transmission

File: src/kuka-lwr/lwr_description/model/kuka_lwr.transmission.xacro (robot description, xacro)
@@ -3,4 +3,5 @@
 	<xacro:property name="Interface10" value="PositionJointInterface"/>
 	<xacro:property name="Interface30" value="EffortJointInterface"/>
+	<xacro:property name="Interface50" value="VelocityJointInterface"/>
 	<xacro:macro name="kuka_lwr_transmission" params="name">
 		<transmission name="${name}_a1_trans">
